File: Miniscope-V4-Ephys-System/Connector-Interface.sch (KiCad schematic (older format))
At the start: 12 parts, among them J10 Conn_01x01, J11 Conn_01x01, J12 Conn_01x01, J13 Conn_01x01, J2 Conn_01x01, J3 Conn_01x01, J4 Conn_01x01, J5 Conn_01x01, J6 Conn_01x01, J7 Conn_01x01, J8 Conn_01x01, J9 Conn_01x01

Commit message: Switch to female slimstack and reorder pins to batch 32ch silicon probe connector
Parts:
- J11, J13, J3, J5, J7, J9: footprint .Connector:Spring_2306654_3 -> .Connector:Conn_1x1_250x750_Pad
Changed lines of the file:
@@
 F 0 "J3" H 5305 3521 50  0000 L CNN
 F 1 "Conn_01x01" H 5305 3521 50  0001 L CNN
-F 2 ".Connector:Spring_2306654_3" H 5225 3525 50  0001 C CNN
+F 2 ".Connector:Conn_1x1_250x750_Pad" H 5225 3525 50  0001 C CNN
 F 3 "~" H 5225 3525 50  0001 C CNN
 	1    5225 3525
@@
 F 0 "J5" H 5305 3621 50  0000 L CNN
 F 1 "Conn_01x01" H 5305 3621 50  0001 L CNN
-F 2 ".Connector:Spring_2306654_3" H 5225 3625 50  0001 C CNN
+F 2 ".Connector:Conn_1x1_250x750_Pad" H 5225 3625 50  0001 C CNN
 F 3 "~" H 5225 3625 50  0001 C CNN
 	1    5225 3625
@@
 F 0 "J7" H 5305 3721 50  0000 L CNN
 F 1 "Conn_01x01" H 5305 3721 50  0001 L CNN
-F 2 ".Connector:Spring_2306654_3" H 5225 3725 50  0001 C CNN
+F 2 ".Connector:Conn_1x1_250x750_Pad" H 5225 3725 50  0001 C CNN
 F 3 "~" H 5225 3725 50  0001 C CNN
 	1    5225 3725
@@
 F 0 "J9" H 5305 3821 50  0000 L CNN
 F 1 "Conn_01x01" H 5305 3821 50  0001 L CNN
-F 2 ".Connector:Spring_2306654_3" H 5225 3825 50  0001 C CNN
+F 2 ".Connector:Conn_1x1_250x750_Pad" H 5225 3825 50  0001 C CNN
 F 3 "~" H 5225 3825 50  0001 C CNN
 	1    5225 3825
@@
 F 0 "J11" H 5305 3921 50  0000 L CNN
 F 1 "Conn_01x01" H 5305 3921 50  0001 L CNN
-F 2 ".Connector:Spring_2306654_3" H 5225 3925 50  0001 C CNN
+F 2 ".Connector:Conn_1x1_250x750_Pad" H 5225 3925 50  0001 C CNN
 F 3 "~" H 5225 3925 50  0001 C CNN
 	1    5225 3925
@@
 F 0 "J13" H 5305 4021 50  0000 L CNN
 F 1 "Conn_01x01" H 5305 4021 50  0001 L CNN
-F 2 ".Connector:Spring_2306654_3" H 5225 4025 50  0001 C CNN
+F 2 ".Connector:Conn_1x1_250x750_Pad" H 5225 4025 50  0001 C CNN
 F 3 "~" H 5225 4025 50  0001 C CNN
 	1    5225 4025
